File: KiCad/sch_usb-c_connector.kicad_sch (KiCad schematic)
At the start: 6 parts, among them J1 USB-C-16P (USB 2.0 only), U2 USBLC6-4SC6

Commit message: Update BoM
Update components with full description and Digikey P/N.
Parts:
- C3: Digikey_PN (none) -> 399-C0603C104K4RACTUCT-ND
- J1: Digikey_PN (none) -> 2073-USB4105-GF-A-120CT-ND
- R2, R3: Digikey_PN (none) -> 541-4030-1-ND
- U2: Digikey_PN (none) -> 497-4492-1-ND
Changed lines of the file:
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@@
+			)
+		)
+		(property "Sim.Device" ""
+			(at 121.92 52.07 0)
+			(effects
+				(font
+					(size 1.27 1.27)
+				)
+			)
+		)
+		(property "Sim.Library" ""
+			(at 121.92 52.07 0)
+			(effects
+				(font
+					(size 1.27 1.27)
+				)
+			)
+		)
+		(property "Sim.Name" ""
+			(at 121.92 52.07 0)
+			(effects
+				(font
+					(size 1.27 1.27)
+				)
+			)
+		)
+		(property "Sim.Params" ""
+			(at 121.92 52.07 0)
+			(effects
+				(font
+					(size 1.27 1.27)
+				)
+			)
+		)
+		(property "Sim.Pins" ""
+			(at 121.92 52.07 0)
+			(effects
+				(font
+					(size 1.27 1.27)
+				)
 			)
 		)
@@
 			)
 		)
-		(property "Description" "Very low capacitance ESD protection diode, 4 data-line, SOT-23-6"
+		(property "Description" "17V Clamp 5A (8/20µs) Ipp Tvs Diode Surface Mount SOT-23-6"
 			(at 204.47 62.23 0)
 			(effects
@@
 				)
 				(hide yes)
+			)
+		)
+		(property "Sim.Device" ""
+			(at 204.47 62.23 0)
+			(effects
+				(font
+					(size 1.27 1.27)
+				)
+				(hide yes)
+			)
+		)
+		(property "Sim.Library" ""
+			(at 204.47 62.23 0)
+			(effects
+				(font
+					(size 1.27 1.27)
+				)
+				(hide yes)
+			)
+		)
+		(property "Sim.Name" ""
+			(at 204.47 62.23 0)
+			(effects
+				(font
+					(size 1.27 1.27)
+				)
+				(hide yes)
+			)
+		)
+		(property "Sim.Params" ""
+			(at 204.47 62.23 0)
+			(effects
+				(font
+					(size 1.27 1.27)
+				)
+				(hide yes)
+			)
+		)
+		(property "Supplier" ""
+			(at 204.47 62.23 0)
+			(effects
+				(font
+					(size 1.27 1.27)
+				)
+				(hide yes)
+			)
+		)
+		(property "Digikey_PN" "497-4492-1-ND"
+			(at 204.47 62.23 0)
+			(effects
+				(font
+					(size 1.27 1.27)
+				)
+				(hide yes)
+			)
+		)
+		(property "Sim.Pins" ""
+			(at 204.47 62.23 0)
+			(effects
+				(font
+					(size 1.27 1.27)
+				)
 			)
 		)
@@
 			)
 		)
-		(property "Description" "USB 2.0-only 16P Type-C Receptacle connector"
+		(property "Description" "USB-C (USB TYPE-C) USB 2.0 Receptacle Connector 24 (16+8 Dummy) Position Surface Mount, Right Angle; Through Hole"
 			(at 96.52 67.31 0)
 			(effects
@@
 			)
 		)
-		(property "Digikey_PN" ""
+		(property "Digikey_PN" "2073-USB4105-GF-A-120CT-ND"
 			(at 96.52 67.31 0)
 			(effects
@@
 			)
 		)
-		(property "Description" "Resistor"
+		(property "Description" "5.1 kOhms ±1% 0.1W, 1/10W Chip Resistor 0603 (1608 Metric) Thick Film"
 			(at 121.92 57.15 0)
 			(effects
@@
 			)
 		)
-		(property "Digikey_PN" ""
+		(property "Digikey_PN" "541-4030-1-ND"
 			(at 121.92 57.15 0)
 			(effects
@@
 				)
 				(hide yes)
+			)
+		)
+		(property "Sim.Device" ""
+			(at 121.92 57.15 0)
+			(effects
+				(font
+					(size 1.27 1.27)
+				)
+			)
+		)
+		(property "Sim.Library" ""
+			(at 121.92 57.15 0)
+			(effects
+				(font
+					(size 1.27 1.27)
+				)
+			)
+		)
+		(property "Sim.Name" ""
+			(at 121.92 57.15 0)
+			(effects
+				(font
+					(size 1.27 1.27)
+				)
+			)
+		)
+		(property "Sim.Params" ""
+			(at 121.92 57.15 0)
+			(effects
+				(font
+					(size 1.27 1.27)
+				)
+			)
+		)
+		(property "Sim.Pins" ""
+			(at 121.92 57.15 0)
+			(effects
+				(font
+					(size 1.27 1.27)
+				)
 			)
 		)
@@
 			)
 		)
-		(property "Description" "Unpolarized capacitor, small symbol"
+		(property "Description" "CAP CER 100nF (0.1uF) 16V X7R 0603"
 			(at 214.63 55.88 0)
 			(effects
@@
 			)
 		)
-		(property "Digikey_PN" ""
+		(property "Digikey_PN" "399-C0603C104K4RACTUCT-ND"
 			(at 214.63 55.88 0)
 			(effects
@@
 				)
 				(hide yes)
+			)
+		)
+		(property "Sim.Pins" ""
+			(at 214.63 55.88 0)
+			(effects
+				(font
+					(size 1.27 1.27)
+				)
 			)
 		)
@@
 			)
 		)
-		(property "Description" "Resistor"
+		(property "Description" "5.1 kOhms ±1% 0.1W, 1/10W Chip Resistor 0603 (1608 Metric) Thick Film"
 			(at 121.92 59.69 0)
 			(effects
@@
 			)
 		)
-		(property "Digikey_PN" ""
+		(property "Digikey_PN" "541-4030-1-ND"
 			(at 121.92 59.69 0)
 			(effects
@@
 			)
 		)
+		(property "Sim.Device" ""
+			(at 121.92 59.69 0)
+			(effects
+				(font
+					(size 1.27 1.27)
+				)
+			)
+		)
+		(property "Sim.Library" ""
+			(at 121.92 59.69 0)
+			(effects
+				(font
+					(size 1.27 1.27)
+				)
+			)
+		)
+		(property "Sim.Name" ""
+			(at 121.92 59.69 0)
+			(effects
+				(font
+					(size 1.27 1.27)
+				)
+			)
+		)
+		(property "Sim.Params" ""
+			(at 121.92 59.69 0)
+			(effects
+				(font
+					(size 1.27 1.27)
+				)
+			)
+		)
+		(property "Sim.Pins" ""
+			(at 121.92 59.69 0)
+			(effects
+				(font
+					(size 1.27 1.27)
+				)
+			)
+		)

Commit message: Update BOM and general tidy-up
Include DigiKey cut-tape components and add flag to indicate own stocked items. Remove files that aren't part of the sharable project (KiCad 9 embeds), Remove empty/irrelevant folders.
Parts:
- C3: Stocked (none) -> Yes
Changed lines of the file:
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@@
 			)
 		)
-		(property "Sim.Pins" ""
+		(property "Stocked" "Yes"
 			(at 214.63 55.88 0)
 			(effects
@@
 					(size 1.27 1.27)
 				)
+				(hide yes)
 			)
 		)
+		(property "Silk" ""
+			(at 214.63 55.88 0)
+			(effects
+				(font
+					(size 1.27 1.27)
+				)
+				(hide yes)
+			)
+		)
